File: hardware/ip_simple.brd (EAGLE design)
At the start: 28 x 31 mm, 32 parts, among them Q4 irml9301, Q7 irml9301, T1 BC846, T3 BC846, Y1 32768Hz CFPX-217 12.5pF

Commit message: sent to manufacturer
Parts:
- moved JP1 5.10 mm to (1.80, 27.7), turned to 270 degrees
- moved U$7 0.81 mm to (18.8, 27.6)
- moved G1 0.20 mm to (14.4, 15.4)
- moved JP2 0.20 mm to (1.80, 2.30)
Routing:
- net AVP: track 5.88 -> 9.55 mm
- net TEST: track 18.7 -> 20.1 mm
- net RST: track 20.3 -> 21.3 mm
- net GND: vias 15 -> 17

Commit message: rev 2
Parts:
- removed C17: 100nF, rcl:C0805
- removed JP2: prog, SparkFun-Connectors:1X06-SIP_LOCK
- added C1: 100nF, rcl:C0805
- added U$2: MOLEX_6VERTICAL, Simplex-Connectors:0530470610
- moved R22 18.7 mm to (23.8, 20.9), turned to 0 degrees
- moved R24 14.5 mm to (23.8, 18.8)
- moved U$7 12.5 mm to (6.30, 27.7), flipped to the bottom
- moved C18 10.3 mm to (23.8, 16.7)
- moved C24 6.21 mm to (24.9, 5.20), turned to 270 degrees
- moved R21 6.00 mm to (8.90, 20.9)
- moved R19 5.20 mm to (18.6, 20.9)
- moved C23 4.77 mm to (22.7, 5.20), turned to 270 degrees
- moved D1 4.74 mm to (13.1, 24.4), turned to 90 degrees
- moved C10 4.40 mm to (23.8, 14.6)
- moved R2 3.09 mm to (13.6, 20.4)
- moved R20 3.09 mm to (13.6, 16.2), turned to 0 degrees
- moved Y1 2.55 mm to (23.8, 8.40), turned to 180 degrees
- moved C8 2.30 mm to (23.8, 12.5)
- moved Q7 2.06 mm to (8.90, 24.4)
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Connections:
- removed net P6.2: C18.1, R22.2, R24.1, U$1.3
- new net P1.1: C18.1, R22.2, R24.1, U$1.15
- net GND: now also C1.2, U$2.1; no longer C17.1, JP2.1
- net N$4: now also C1.1
- net RST: now also U$2.2; no longer JP2.2
- net RX: now also U$2.5; no longer JP2.5
- net TEST: now also U$2.3; no longer JP2.3
- net TX: now also U$2.6; no longer JP2.6
- net VCC: now also U$2.4; no longer C17.2, JP2.4
Routing:
- net PX: track 55.0 -> 29.1 mm, vias 5 -> 3
- net GND: track 31.7 -> 16.2 mm, vias 17 -> 20
- net P1.1: track 0.00 -> 14.4 mm
- net P6.2: track 8.87 -> 0.00 mm
- net N$31: track 12.5 -> 5.85 mm, vias 2 -> 0
- net VCC: track 55.8 -> 50.3 mm
- net AVP: track 9.55 -> 14.7 mm
- net TALK_EN: track 7.48 -> 2.81 mm
- net N$3: track 2.72 -> 7.10 mm
- net N$25: track 6.09 -> 10.2 mm
- net N$5: track 3.77 -> 7.49 mm
- net OPEN_EN: track 3.63 -> 6.67 mm
- net N$6: track 9.14 -> 6.11 mm
- net N$32: track 6.76 -> 4.60 mm
- net N$28: track 6.36 -> 4.60 mm
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Other:
- board text added: "ip rev 2.0 201312"
- board text removed: "ip rev 1.0 201311"

Commit message: cleanup for unused pins
Parts:
- removed C11: 220nF, rcl:C0805
- removed U$2: MOLEX_6VERTICAL, Simplex-Connectors:0530470610
- added X1: MOLEX_6VERTICAL, Simplex-Connectors:0530470610
Connections:
- removed net 41: U$1.41
- removed net N$7: C11.1, U$1.43
- new net 43: U$1.43
- net GND: now also U$1.39, U$1.41, X1.1; no longer C11.2, U$2.1
- net RST: now also X1.2; no longer U$2.2
- net RX: now also X1.5; no longer U$2.5
- net TEST: now also X1.3; no longer U$2.3
- net TX: now also X1.6; no longer U$2.6
- net VCC: now also X1.4; no longer U$2.4
Routing:
- net N$7: track 5.74 -> 0.00 mm
- net GND: track 16.2 -> 19.3 mm
Changed lines of the file:
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@@
 <text x="1" y="13.6" size="0.8128" layer="108" font="vector" ratio="15">gnd</text>
 <text x="27.3" y="26.2" size="0.8128" layer="109" font="vector" ratio="15" rot="MR270">http://github.com/rodan/interphone</text>
-<text x="23.7" y="16.8" size="0.8128" layer="109" font="vector" ratio="15" rot="MR270">ip rev 2.0 201312</text>
+<text x="23.6" y="21.4" size="0.8128" layer="109" font="vector" ratio="15" rot="MR270">ip rev 2.0 201312</text>
 </plain>
 <attributes>
@@
 <element name="U$1" library="TI_MSP430_v16" package="PT48" value="F55[0/1]X---PT48" x="14.4" y="9.3" rot="R180"/>
 <element name="C10" library="rcl" package="C0805" value="470nF" x="23.8" y="14.6"/>
-<element name="C11" library="rcl" package="C0805" value="220nF" x="19.3" y="2.2"/>
 <element name="R6" library="rcl" package="R0805W" value="4.7k" x="5.7" y="9.9"/>
 <element name="R7" library="rcl" package="R0805W" value="4.7k" x="5.7" y="12"/>
@@
 <element name="R2" library="rcl" package="R0805W" value="2k2" x="13.6" y="20.4" rot="R180"/>
 <element name="JP1" library="SparkFun-Connectors" package="1X03" value="interphone" x="2.3" y="27.7" rot="R270"/>
-<element name="U$2" library="Simplex-Connectors" package="0530470610" value="MOLEX_6VERTICAL" x="2.2" y="4.9" rot="R90"/>
 <element name="C1" library="rcl" package="C0805" value="100nF" x="18.6" y="27.7"/>
+<element name="X1" library="Simplex-Connectors" package="0530470610" value="MOLEX_6VERTICAL" x="2.3" y="4.9" rot="R90"/>
 </elements>
 <signals>
 <signal name="GND">
 <contactref element="U$1" pad="12"/>
-<contactref element="C11" pad="2"/>
 <contactref element="U$1" pad="37"/>
 <contactref element="C23" pad="2"/>
@@
 <wire x1="18.7" y1="11.05" x2="20.05" y2="11.05" width="0.3048" layer="1"/>
 <polygon width="0.3048" layer="1" isolate="0.4064">
-<vertex x="0.4" y="31.7"/>
+<vertex x="0" y="31"/>
 <vertex x="0" y="0"/>
-<vertex x="28.3" y="0"/>
-<vertex x="28.3" y="31.7"/>
+<vertex x="28" y="0"/>
+<vertex x="28" y="31"/>
 </polygon>
 <polygon width="0.3048" layer="16" isolate="0.4064">
-<vertex x="0.4" y="31.8"/>
+<vertex x="0" y="31"/>
 <vertex x="0" y="0"/>
-<vertex x="27.6" y="0"/>
-<vertex x="27.6" y="31.8"/>
+<vertex x="28" y="0"/>
+<vertex x="28" y="31"/>
 </polygon>
 <via x="24.7" y="23.5" extent="1-16" drill="0.4"/>
@@
 <via x="6.5" y="18.5" extent="1-16" drill="0.4"/>
 <via x="1.6" y="20.7" extent="1-16" drill="0.4"/>
-<contactref element="U$2" pad="1"/>
 <wire x1="11.65" y1="5" x2="11" y2="5" width="0.3048" layer="1"/>
 <wire x1="20.05" y1="11.05" x2="20.3" y2="11.3" width="0.3048" layer="1"/>
@@
 <wire x1="16.65" y1="12.05" x2="16.2" y2="11.6" width="0.3048" layer="1"/>
 <contactref element="C1" pad="2"/>
+<contactref element="U$1" pad="41"/>
+<contactref element="U$1" pad="39"/>
+<wire x1="13.65" y1="5" x2="13.65" y2="6.45" width="0.3048" layer="1"/>
+<wire x1="13.65" y1="6.45" x2="13.7" y2="6.5" width="0.3048" layer="1"/>
+<wire x1="12.65" y1="5" x2="12.65" y2="6.55" width="0.3048" layer="1"/>
+<wire x1="12.65" y1="6.55" x2="12.7" y2="6.6" width="0.3048" layer="1"/>
+<contactref element="X1" pad="1"/>
 </signal>
 <signal name="N$6">
@@
 <wire x1="17.15" y1="13.6" x2="21.85" y2="13.6" width="0.3048" layer="1"/>
 <wire x1="21.85" y1="13.6" x2="22.85" y2="14.6" width="0.3048" layer="1"/>
-</signal>
-<signal name="N$7">
-<contactref element="U$1" pad="43"/>
-<contactref element="C11" pad="1"/>
-<wire x1="14.65" y1="5" x2="14.65" y2="3.95" width="0.3048" layer="1"/>
-<wire x1="14.65" y1="3.95" x2="14.8" y2="3.8" width="0.3048" layer="1"/>
-<wire x1="14.8" y1="3.8" x2="16" y2="3.8" width="0.3048" layer="1"/>
-<wire x1="16" y1="3.8" x2="17" y2="2.8" width="0.3048" layer="1"/>
-<wire x1="17" y1="2.8" x2="18.2" y2="2.8" width="0.3048" layer="1"/>
-<wire x1="18.2" y1="2.8" x2="18.35" y2="2.65" width="0.3048" layer="1"/>
-<wire x1="18.35" y1="2.65" x2="18.35" y2="2.2" width="0.3048" layer="1"/>
 </signal>
 <signal name="N$11">
@@
 <signal name="RX">
 <contactref element="R6" pad="1"/>
-<contactref element="U$2" pad="5"/>
-<wire x1="4.6475" y1="9.9" x2="2.2" y2="9.9" width="0.3048" layer="1"/>
+<contactref element="X1" pad="5"/>
+<wire x1="4.6475" y1="9.9" x2="2.3" y2="9.9" width="0.3048" layer="1"/>
 </signal>
 <signal name="TX">
 <contactref element="R7" pad="1"/>
-<contactref element="U$2" pad="6"/>
-<wire x1="3.4975" y1="11.15" x2="2.2" y2="11.15" width="0.3048" layer="1"/>
 <wire x1="3.4975" y1="11.15" x2="4.3475" y2="12" width="0.3048" layer="1"/>
 <wire x1="4.3475" y1="12" x2="4.6475" y2="12" width="0.3048" layer="1"/>
+<contactref element="X1" pad="6"/>
+<wire x1="3.4975" y1="11.15" x2="2.3" y2="11.15" width="0.3048" layer="1"/>
 </signal>
 <signal name="N$25">
@@
 <wire x1="8.4" y1="5.2" x2="7.9" y2="4.7" width="0.3048" layer="16"/>
 <wire x1="7.9" y1="4.7" x2="7.8" y2="4.7" width="0.3048" layer="16"/>
-<contactref element="U$2" pad="4"/>
 <wire x1="19.65" y1="11.55" x2="20.5" y2="12.4" width="0.3048" layer="1"/>
 <wire x1="20.5" y1="12.4" x2="22.75" y2="12.4" width="0.3048" layer="1"/>
 <wire x1="22.75" y1="12.4" x2="22.85" y2="12.5" width="0.3048" layer="1"/>
 <wire x1="5.4" y1="8.5" x2="5.25" y2="8.65" width="0.3048" layer="1"/>
-<wire x1="5.25" y1="8.65" x2="2.2" y2="8.65" width="0.3048" layer="1"/>
 <wire x1="6.65" y1="14.1" x2="6.75" y2="14.2" width="0.3048" layer="1"/>
 <wire x1="6.75" y1="14.2" x2="9.5" y2="14.2" width="0.3048" layer="1"/>
@@
 <wire x1="13.1" y1="1.63" x2="13.1" y2="1.77" width="0.3048" layer="16"/>
 <wire x1="13.1" y1="1.77" x2="13.13" y2="1.8" width="0.3048" layer="16"/>
+<contactref element="X1" pad="4"/>
+<wire x1="5.25" y1="8.65" x2="2.3" y2="8.65" width="0.3048" layer="1"/>
 </signal>
 <signal name="LED">
@@
 <wire x1="18.7" y1="4" x2="18.1" y2="4.6" width="0.3048" layer="16"/>
 <wire x1="18.1" y1="4.6" x2="18.1" y2="4.8" width="0.3048" layer="16"/>
-<contactref element="U$2" pad="2"/>
 <wire x1="4.6475" y1="5.1" x2="3.4" y2="6.1" width="0.3048" layer="1"/>
-<wire x1="3.4" y1="6.1" x2="2.2" y2="6.15" width="0.3048" layer="1"/>
+<contactref element="X1" pad="2"/>
+<wire x1="3.4" y1="6.1" x2="2.3" y2="6.1" width="0.3048" layer="1"/>
+<wire x1="2.3" y1="6.1" x2="2.3" y2="6.15" width="0.3048" layer="1"/>
 </signal>
 <signal name="TEST">
@@
 <wire x1="15.6" y1="5.1" x2="17" y2="3.7" width="0.3048" layer="16"/>
 <wire x1="17" y1="3.7" x2="17.8" y2="3.7" width="0.3048" layer="16"/>
-<contactref element="U$2" pad="3"/>
 <wire x1="4.6475" y1="7.2" x2="4.6475" y2="6.7525" width="0.3048" layer="1"/>
 <wire x1="4.6475" y1="6.7525" x2="5.2" y2="6.2" width="0.3048" layer="1"/>
@@
 <wire x1="8.1" y1="6.2" x2="8.2" y2="6.3" width="0.3048" layer="1"/>
 <wire x1="4.6475" y1="7.2" x2="4.4475" y2="7.4" width="0.3048" layer="1"/>
-<wire x1="4.4475" y1="7.4" x2="2.2" y2="7.4" width="0.3048" layer="1"/>
+<contactref element="X1" pad="3"/>
+<wire x1="4.4475" y1="7.4" x2="2.3" y2="7.4" width="0.3048" layer="1"/>
 </signal>
 <signal name="OPEN_EN">
@@
 <contactref element="U$1" pad="46"/>
 </signal>
-<signal name="41">
-<contactref element="U$1" pad="41"/>
-</signal>
 <signal name="AVP">
 <contactref element="D1" pad="C"/>
@@
 <wire x1="23.6525" y1="19.7" x2="24.8525" y2="20.9" width="0.3048" layer="1"/>
 </signal>
+<signal name="43">
+<contactref element="U$1" pad="43"/>
+</signal>
 </signals>
